Commit message: Updated URDF to reflect change of joint_1 type

File: src/adele_urdf_1/urdf/adele_urdf_1.urdf (robot description, URDF)
Before this commit: robot adele_urdf_1, 10 links, 9 joints
Joints:
- joint joint_1: limit (none) -> lower=-3.49066 upper=3.49066 effort=0 velocity=0; type continuous -> revolute
