Commit message: Updated joint_6 limits

File: src/adele_urdf_2/urdf/adele_urdf_2.urdf (robot description, URDF)
Before this commit: robot adele_urdf_2, 7 links, 6 joints
Joints:
- joint Joint_6: limit lower=-3.14 upper=3.14 effort=0 velocity=125.7 -> lower=-0.785398 upper=0.785398 effort=0 velocity=125.7
